Commit message: load all controller normal

File: a1_description/xacro/a1.ros2_control.xacro (robot description, xacro)
@@ -11,14 +11,37 @@
         <param name="max">0.5</param>
       </command_interface>
-      <command_interface name="Kp"/>
-      <command_interface name="Kd"/>
-      <command_interface name="effort_limit"/>
       <state_interface name="position"/>
       <state_interface name="velocity"/>
       <state_interface name="effort"/>
-      <state_interface name="coil_resistance"/>
-      <state_interface name="timestamp"/>
     </joint>
     <joint name="FL_thigh_joint">
+      <command_interface name="effort">
+        <param name="min">-0.5</param>
+        <param name="max">0.5</param>
+      </command_interface>
+      <state_interface name="position"/>
+      <state_interface name="velocity"/>
+      <state_interface name="effort"/>
+    </joint>
+    <joint name="FL_calf_joint">
+      <command_interface name="effort">
+        <param name="min">-0.5</param>
+        <param name="max">0.5</param>
+      </command_interface>
+      <state_interface name="position"/>
+      <state_interface name="velocity"/>
+      <state_interface name="effort"/>
+    </joint>
+    <!--front right leg-->
+    <joint name="FR_hip_joint">
+      <command_interface name="effort">
+        <param name="min">-1</param>
+        <param name="max">1</param>
+      </command_interface>
+      <state_interface name="position"/>
+      <state_interface name="velocity"/>
+      <state_interface name="effort"/>
+    </joint>
+    <joint name="FR_thigh_joint">
       <command_interface name="effort">
         <param name="min">-0.5</param>
@@ -31,89 +54,14 @@
       <state_interface name="velocity"/>
       <state_interface name="effort"/>
-      <state_interface name="coil_resistance"/>
-      <state_interface name="timestamp"/>
     </joint>
-    <joint name="FL_calf_joint">
+    <joint name="FR_calf_joint">
       <command_interface name="effort">
         <param name="min">-0.5</param>
         <param name="max">0.5</param>
       </command_interface>
-      <command_interface name="Kp"/>
-      <command_interface name="Kd"/>
-      <command_interface name="effort_limit"/>
       <state_interface name="position"/>
       <state_interface name="velocity"/>
       <state_interface name="effort"/>
-      <state_interface name="coil_resistance"/>
-      <state_interface name="contact_information"/>
-      <state_interface name="timestamp"/>
     </joint>
-    <!--front right leg-->
-    <!--<joint name="FR_hip_joint">
-      <command_interface name="position">
-        <param name="min">-1</param>
-        <param name="max">1</param>
-      </command_interface>
-      <command_interface name="velocity">
-        <param name="min">-1</param>
-        <param name="max">1</param>
-      </command_interface>
-      <command_interface name="effort">
-        <param name="min">-0.5</param>
-        <param name="max">0.5</param>
-      <command_interface name="Kp"/>
-      <command_interface name="Kd"/>
-      <command_interface name="effort_limit"/>
-      <state_interface name="position"/>
-      <state_interface name="velocity"/>
-      <state_interface name="effort"/>
-      <state_interface name="coil_resistance"/>
-      <state_interface name="timestamp"/>
-    </joint>
-    <joint name="FR_thigh_joint">
-      <command_interface name="position">
-        <param name="min">-1</param>
-        <param name="max">1</param>
-      </command_interface>
-      <command_interface name="velocity">
-        <param name="min">-1</param>
-        <param name="max">1</param>
-      </command_interface>
-      <command_interface name="effort">
-        <param name="min">-0.5</param>
-        <param name="max">0.5</param>
-      </command_interface>
-      <command_interface name="Kp"/>
-      <command_interface name="Kd"/>
-      <command_interface name="effort_limit"/>
-      <state_interface name="position"/>
-      <state_interface name="velocity"/>
-      <state_interface name="effort"/>
-      <state_interface name="coil_resistance"/>
-      <state_interface name="timestamp"/>
-    </joint>
-    <joint name="FR_calf_joint">
-      <command_interface name="position">
-        <param name="min">-1</param>
-        <param name="max">1</param>
-      </command_interface>
-      <command_interface name="velocity">
-        <param name="min">-1</param>
-        <param name="max">1</param>
-      </command_interface>
-      <command_interface name="effort">
-        <param name="min">-0.5</param>
-        <param name="max">0.5</param>
-      </command_interface>
-      <command_interface name="Kp"/>
-      <command_interface name="Kd"/>
-      <command_interface name="effort_limit"/>
-      <state_interface name="position"/>
-      <state_interface name="velocity"/>
-      <state_interface name="effort"/>
-      <state_interface name="coil_resistance"/>
-      <state_interface name="contact_information"/>
-      <state_interface name="timestamp"/>
-    </joint>-->
     <!--left leg-->
     <joint name="RL_hip_joint">
@@ -122,12 +70,7 @@
         <param name="max">0.5</param>
       </command_interface>
-      <command_interface name="Kp"/>
-      <command_interface name="Kd"/>
-      <command_interface name="effort_limit"/>
       <state_interface name="position"/>
       <state_interface name="velocity"/>
       <state_interface name="effort"/>
-      <state_interface name="coil_resistance"/>
-      <state_interface name="timestamp"/>
     </joint>
     <joint name="RL_thigh_joint">
@@ -136,102 +79,45 @@
         <param name="max">0.5</param>
       </command_interface>
-      <command_interface name="Kp"/>
-      <command_interface name="Kd"/>
-      <command_interface name="effort_limit"/>
       <state_interface name="position"/>
       <state_interface name="velocity"/>
       <state_interface name="effort"/>
-      <state_interface name="coil_resistance"/>
-      <state_interface name="timestamp"/>
     </joint>
-    <!--<joint name="RL_calf_joint">
-      <command_interface name="position">
-        <param name="min">-1</param>
-        <param name="max">1</param>
-      </command_interface>
-      <command_interface name="velocity">
-        <param name="min">-1</param>
-        <param name="max">1</param>
-      </command_interface>
-      <command_interface name="effort">
-        <param name="min">-0.5</param>
-        <param name="max">0.5</param>
-      <command_interface name="Kp"/>
-      <command_interface name="Kd"/>
-      <command_interface name="effort_limit"/>
-      <state_interface name="position"/>
-      <state_interface name="velocity"/>
-      <state_interface name="effort"/>
-      <state_interface name="coil_resistance"/>
-      <state_interface name="contact_information"/>
-      <state_interface name="timestamp"/>
-    </joint>-->
-    <!--right leg-->
-    <!--<joint name="RR_hip_joint">
-      <command_interface name="position">
-        <param name="min">-1</param>
-        <param name="max">1</param>
-      </command_interface>
-      <command_interface name="velocity">
-        <param name="min">-1</param>
-        <param name="max">1</param>
-      </command_interface>
+    <joint name="RL_calf_joint">
       <command_interface name="effort">
         <param name="min">-0.5</param>
         <param name="max">0.5</param>
       </command_interface>
-      <command_interface name="Kp"/>
-      <command_interface name="Kd"/>
-      <command_interface name="effort_limit"/>
       <state_interface name="position"/>
       <state_interface name="velocity"/>
       <state_interface name="effort"/>
-      <state_interface name="coil_resistance"/>
-      <state_interface name="timestamp"/>
     </joint>
-    <joint name="RR_thigh_joint">
-      <command_interface name="position">
-        <param name="min">-1</param>
-        <param name="max">1</param>
-      </command_interface>
-      <command_interface name="velocity">
-        <param name="min">-1</param>
-        <param name="max">1</param>
-      </command_interface>
+    <!--right leg-->
+    <joint name="RR_hip_joint">
       <command_interface name="effort">
         <param name="min">-0.5</param>
         <param name="max">0.5</param>
       </command_interface>
-      <command_interface name="Kp"/>
-      <command_interface name="Kd"/>
-      <command_interface name="effort_limit"/>
       <state_interface name="position"/>
       <state_interface name="velocity"/>
       <state_interface name="effort"/>
-      <state_interface name="coil_resistance"/>
-      <state_interface name="timestamp"/>
     </joint>
-    <joint name="RR_calf_joint">
-      <command_interface name="position">
-        <param name="min">-1</param>
-        <param name="max">1</param>
-      </command_interface>
-      <command_interface name="velocity">
-        <param name="min">-1</param>
-        <param name="max">1</param>
-      </command_interface>
+    <joint name="RR_thigh_joint">
       <command_interface name="effort">
         <param name="min">-0.5</param>
         <param name="max">0.5</param>
-      <command_interface name="Kp"/>
-      <command_interface name="Kd"/>
-      <command_interface name="effort_limit"/>
+      </command_interface>
       <state_interface name="position"/>
       <state_interface name="velocity"/>
       <state_interface name="effort"/>
-      <state_interface name="coil_resistance"/>
-      <state_interface name="contact_information"/>
-      <state_interface name="timestamp"/>
-    </joint>-->
+    </joint>
+    <joint name="RR_calf_joint">
+      <command_interface name="effort">
+        <param name="min">-0.5</param>
+        <param name="max">0.5</param>
+      </command_interface>
+      <state_interface name="position"/>
+      <state_interface name="velocity"/>
+      <state_interface name="effort"/>
+    </joint>
   </ros2_control>
 </robot>

Commit message: message

File: a1_description/xacro/a1.ros2_control.xacro (robot description, xacro)
@@ -7,5 +7,42 @@
     <!--left front leg hip-->
     <joint name="FL_hip_joint">
-      <command_interface name="effort">
+      <command_interface name="velocity">
+        <param name="min">-0.5</param>
+        <param name="max">0.5</param>
+      </command_interface>
+      <state_interface name="position"/>
+      <state_interface name="velocity"/>
+      <state_interface name="effort"/>
+    </joint>
+    <joint name="FL_thigh_joint">
+      <command_interface name="velocity">
+        <param name="min">-0.5</param>
+        <param name="max">0.5</param>
+      </command_interface>
+      <state_interface name="position"/>
+      <state_interface name="velocity"/>
+      <state_interface name="effort"/>
+    </joint>
+    <joint name="FL_calf_joint">
+      <command_interface name="velocity">
+        <param name="min">-0.5</param>
+        <param name="max">0.5</param>
+      </command_interface>
+      <state_interface name="position"/>
+      <state_interface name="velocity"/>
+      <state_interface name="effort"/>
+    </joint>
+    <!--front right leg-->
+    <joint name="FR_hip_joint">
+      <command_interface name="velocity">
+        <param name="min">-1</param>
+        <param name="max">1</param>
+      </command_interface>
+      <state_interface name="position"/>
+      <state_interface name="velocity"/>
+      <state_interface name="effort"/>
+    </joint>
+    <joint name="FR_thigh_joint">
+      <command_interface name="velocity">
         <param name="min">-0.5</param>
         <param name="max">0.5</param>
@@ -17,221 +54,70 @@
       <state_interface name="velocity"/>
       <state_interface name="effort"/>
-      <state_interface name="coil_resistance"/>
-      <state_interface name="timestamp"/>
     </joint>
-    <joint name="FL_thigh_joint">
-      <command_interface name="effort">
+    <joint name="FR_calf_joint">
+      <command_interface name="velocity">
         <param name="min">-0.5</param>
         <param name="max">0.5</param>
       </command_interface>
-      <command_interface name="Kp"/>
-      <command_interface name="Kd"/>
-      <command_interface name="effort_limit"/>
       <state_interface name="position"/>
       <state_interface name="velocity"/>
       <state_interface name="effort"/>
-      <state_interface name="coil_resistance"/>
-      <state_interface name="timestamp"/>
     </joint>
-    <joint name="FL_calf_joint">
-      <command_interface name="effort">
+    <!--left leg-->
+    <joint name="RL_hip_joint">
+      <command_interface name="velocity">
         <param name="min">-0.5</param>
         <param name="max">0.5</param>
       </command_interface>
-      <command_interface name="Kp"/>
-      <command_interface name="Kd"/>
-      <command_interface name="effort_limit"/>
       <state_interface name="position"/>
       <state_interface name="velocity"/>
       <state_interface name="effort"/>
-      <state_interface name="coil_resistance"/>
-      <state_interface name="contact_information"/>
-      <state_interface name="timestamp"/>
     </joint>
-    <!--front right leg-->
-    <!--<joint name="FR_hip_joint">
-      <command_interface name="position">
-        <param name="min">-1</param>
-        <param name="max">1</param>
-      </command_interface>
+    <joint name="RL_thigh_joint">
       <command_interface name="velocity">
-        <param name="min">-1</param>
-        <param name="max">1</param>
-      </command_interface>
-      <command_interface name="effort">
         <param name="min">-0.5</param>
         <param name="max">0.5</param>
-      <command_interface name="Kp"/>
-      <command_interface name="Kd"/>
-      <command_interface name="effort_limit"/>
+      </command_interface>
       <state_interface name="position"/>
       <state_interface name="velocity"/>
       <state_interface name="effort"/>
-      <state_interface name="coil_resistance"/>
-      <state_interface name="timestamp"/>
     </joint>
-    <joint name="FR_thigh_joint">
-      <command_interface name="position">
-        <param name="min">-1</param>
-        <param name="max">1</param>
-      </command_interface>
+    <joint name="RL_calf_joint">
       <command_interface name="velocity">
-        <param name="min">-1</param>
-        <param name="max">1</param>
-      </command_interface>
-      <command_interface name="effort">
         <param name="min">-0.5</param>
         <param name="max">0.5</param>
       </command_interface>
-      <command_interface name="Kp"/>
-      <command_interface name="Kd"/>
-      <command_interface name="effort_limit"/>
       <state_interface name="position"/>
       <state_interface name="velocity"/>
       <state_interface name="effort"/>
-      <state_interface name="coil_resistance"/>
-      <state_interface name="timestamp"/>
     </joint>
-    <joint name="FR_calf_joint">
-      <command_interface name="position">
-        <param name="min">-1</param>
-        <param name="max">1</param>
-      </command_interface>
+    <!--right leg-->
+    <joint name="RR_hip_joint">
       <command_interface name="velocity">
-        <param name="min">-1</param>
-        <param name="max">1</param>
-      </command_interface>
-      <command_interface name="effort">
         <param name="min">-0.5</param>
         <param name="max">0.5</param>
       </command_interface>
-      <command_interface name="Kp"/>
-      <command_interface name="Kd"/>
-      <command_interface name="effort_limit"/>
       <state_interface name="position"/>
       <state_interface name="velocity"/>
       <state_interface name="effort"/>
-      <state_interface name="coil_resistance"/>
-      <state_interface name="contact_information"/>
-      <state_interface name="timestamp"/>
-    </joint>-->
-    <!--left leg-->
-    <joint name="RL_hip_joint">
-      <command_interface name="effort">
+    </joint>
+    <joint name="RR_thigh_joint">
+      <command_interface name="velocity">
         <param name="min">-0.5</param>
         <param name="max">0.5</param>
       </command_interface>
-      <command_interface name="Kp"/>
-      <command_interface name="Kd"/>
-      <command_interface name="effort_limit"/>
       <state_interface name="position"/>
       <state_interface name="velocity"/>
       <state_interface name="effort"/>
-      <state_interface name="coil_resistance"/>
-      <state_interface name="timestamp"/>
     </joint>
-    <joint name="RL_thigh_joint">
-      <command_interface name="effort">
+    <joint name="RR_calf_joint">
+      <command_interface name="velocity">
         <param name="min">-0.5</param>
         <param name="max">0.5</param>
       </command_interface>
-      <command_interface name="Kp"/>
-      <command_interface name="Kd"/>
-      <command_interface name="effort_limit"/>
       <state_interface name="position"/>
       <state_interface name="velocity"/>
       <state_interface name="effort"/>
-      <state_interface name="coil_resistance"/>
-      <state_interface name="timestamp"/>
     </joint>
-    <!--<joint name="RL_calf_joint">
-      <command_interface name="position">
-        <param name="min">-1</param>
-        <param name="max">1</param>
-      </command_interface>
-      <command_interface name="velocity">
-        <param name="min">-1</param>
-        <param name="max">1</param>
-      </command_interface>
-      <command_interface name="effort">
-        <param name="min">-0.5</param>
-        <param name="max">0.5</param>
-      <command_interface name="Kp"/>
-      <command_interface name="Kd"/>
-      <command_interface name="effort_limit"/>
-      <state_interface name="position"/>
-      <state_interface name="velocity"/>
-      <state_interface name="effort"/>
-      <state_interface name="coil_resistance"/>
-      <state_interface name="contact_information"/>
-      <state_interface name="timestamp"/>
-    </joint>-->
-    <!--right leg-->
-    <!--<joint name="RR_hip_joint">
-      <command_interface name="position">
-        <param name="min">-1</param>
-        <param name="max">1</param>
-      </command_interface>
-      <command_interface name="velocity">
-        <param name="min">-1</param>
-        <param name="max">1</param>
-      </command_interface>
-      <command_interface name="effort">
-        <param name="min">-0.5</param>
-        <param name="max">0.5</param>
-      </command_interface>
-      <command_interface name="Kp"/>
-      <command_interface name="Kd"/>
-      <command_interface name="effort_limit"/>
-      <state_interface name="position"/>
-      <state_interface name="velocity"/>
-      <state_interface name="effort"/>
-      <state_interface name="coil_resistance"/>
-      <state_interface name="timestamp"/>
-    </joint>
-    <joint name="RR_thigh_joint">
-      <command_interface name="position">
-        <param name="min">-1</param>
-        <param name="max">1</param>
-      </command_interface>
-      <command_interface name="velocity">
-        <param name="min">-1</param>
-        <param name="max">1</param>
-      </command_interface>
-      <command_interface name="effort">
-        <param name="min">-0.5</param>
-        <param name="max">0.5</param>
-      </command_interface>
-      <command_interface name="Kp"/>
-      <command_interface name="Kd"/>
-      <command_interface name="effort_limit"/>
-      <state_interface name="position"/>
-      <state_interface name="velocity"/>
-      <state_interface name="effort"/>
-      <state_interface name="coil_resistance"/>
-      <state_interface name="timestamp"/>
-    </joint>
-    <joint name="RR_calf_joint">
-      <command_interface name="position">
-        <param name="min">-1</param>
-        <param name="max">1</param>
-      </command_interface>
-      <command_interface name="velocity">
-        <param name="min">-1</param>
-        <param name="max">1</param>
-      </command_interface>
-      <command_interface name="effort">
-        <param name="min">-0.5</param>
-        <param name="max">0.5</param>
-      <command_interface name="Kp"/>
-      <command_interface name="Kd"/>
-      <command_interface name="effort_limit"/>
-      <state_interface name="position"/>
-      <state_interface name="velocity"/>
-      <state_interface name="effort"/>
-      <state_interface name="coil_resistance"/>
-      <state_interface name="contact_information"/>
-      <state_interface name="timestamp"/>
-    </joint>-->
   </ros2_control>
 </robot>
