Commit message: debug undefine symbol

File: a1_description/xacro/gazebo.xacro (robot description, xacro)
@@ -1,19 +1,4 @@
 <?xml version="1.0"?>
 <robot>
-        <!--<ros2_control name="GazeboSystem" type="system">
-    <hardware>
-      <plugin>gazebo_ros2_control/GazeboSystem</plugin>
-    </hardware>
-    <joint name="FL_hip_joint">
-      <command_interface name="position">
-        <param name="min">0</param>
-        <param name="max">0</param>
-      </command_interface>
-      <state_interface name="position"/>
-      <state_interface name="velocity"/>
-      <state_interface name="effort"/>
-        </joint>
-        </ros2_control>-->
-        <!--ros_control plugin -->
     <gazebo>
         <plugin name="gazebo_ros2_control" filename="libgazebo_ros2_control.so">

Commit message: startup imu topic

File: a1_description/xacro/gazebo.xacro (robot description, xacro)
@@ -9,5 +9,4 @@
         </plugin>
     </gazebo>
-    <!-- Show the trajectory of trunk center. -->
     <gazebo>
         <plugin name="3dplot" filename="libLinkPlot3DPlugin.so">
@@ -20,21 +19,13 @@
         </plugin>
     </gazebo>
-    <!-- Show the trajectory of foot. You can add another trajectory about another foot. -->
-    <!-- <gazebo>
-        <plugin name="3dplot" filename="libLinkPlot3DPlugin.so">
-            <frequency>100</frequency>
-            <plot>
-                <link>FL_foot</link>
-                <pose>0 0 0 0 0 0</pose>
-                <material>Gazebo/Green</material>
-            </plot>
+    <gazebo reference="trunk">
+        <plugin filename="libgazebo_ros_force.so" name="gazebo_ros_force">
+            <ros>
+                <namespace>demo</namespace>
+                <argument>/apply_force/trunk:=trunk</argument>
+            </ros>
+            <link_name>trunk</link_name>
         </plugin>
-    </gazebo> -->
-    <!--<gazebo>
-        <plugin filename="libgazebo_ros_force.so" name="gazebo_ros_force">
-            <bodyName>trunk</bodyName>
-            <topicName>/apply_force/trunk</topicName>
-        </plugin>
-    </gazebo>-->
+    </gazebo>
     <gazebo reference="imu_link">
         <gravity>true</gravity>
@@ -45,6 +36,9 @@
             <topic>__default_topic__</topic>
             <plugin filename="libgazebo_ros_imu_sensor.so" name="imu_plugin">
-                <topicName>trunk_imu</topicName>
-                <bodyName>imu_link</bodyName>
+                <ros>
+                    <namespace>/imu</namespace>
+                    <remapping>~/out:=imu_data</remapping>
+                </ros>
+                <link_name>imu_link</link_name>
                 <updateRateHZ>1000.0</updateRateHZ>
                 <gaussianNoise>0.0</gaussianNoise>
